Commit message: Update to fit latest vrx

File: config/sensor_config.xacro (robot description, xacro)
@@ -12,6 +12,6 @@
       <xacro:wamv_camera y="0.2" x="0.75" name="left_camera" P="${radians(15)}" />
       <xacro:wamv_camera y="-0.2" x="0.75" name="right_camera" P="${radians(15)}" />
-    <!-- === wamv_3d_lidar === -->
-      <xacro:wamv_3d_lidar name="velodyne_front" />
+    <!-- === lidar === -->
+      <xacro:lidar name="velodyne_front" />
   </xacro:macro>
 </robot>

File: urdf/ouxt_wamv.urdf (robot description, URDF)
Before this commit: robot WAM-V, 21 links, 20 joints
Links:
- added link dummy_link, mass 180.0; collision box size=0.65 0.2 0.1; collision box size=0.65 0.2 0.1
- link base_link: mass 180.0 -> None; geometry 
Joints:
- added joint dummy_joint: type fixed, parent base_link, child dummy_link

Commit message: Update to add new lidar
The position maked similor as OUXT-Polaris machine.

File: config/sensor_config.xacro (robot description, xacro)
@@ -13,5 +13,6 @@
       <xacro:wamv_camera y="-0.2" x="0.75" name="right_camera" P="${radians(15)}" />
     <!-- === lidar === -->
-      <xacro:lidar name="velodyne_front" />
+      <xacro:lidar x="1.3" z="1.3" name="velodyne_front" />
+      <xacro:lidar x="0.3" name="velodyne_center" />
   </xacro:macro>
 </robot>

File: urdf/ouxt_wamv.urdf (robot description, URDF)
Before this commit: robot WAM-V, 22 links, 21 joints
Links:
- added link velodyne_center_link, mass 1; collision cylinder length=0.075 radius=0.055; visual mesh filename=package://vrx_gazebo/models/3d_lidar/mesh/3d_lidar.dae
- added link velodyne_center_post_arm_link, mass 0.1; collision cylinder length=0.065 radius=0.008; visual mesh filename=package://vrx_gazebo/models/sensor_post/mesh/sensor_post_ar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
- added link velodyne_center_post_link, mass 0.40815; collision cylinder length=0.4535 radius=0.0076; visual cylinder length=0.4535 radius=0.0076
- link velodyne_front_post_link: mass 0.40815 -> -0.04185; geometry collision cylinder length=-0.0465 radius=0.0076; visual cylinder length=-0.0465 radius=0.0076
Joints:
- added joint base_to_velodyne_center_post_joint: type fixed, parent base_link, child velodyne_center_post_link, origin xyz=0.23 0.0 1.52325 rpy=0 0 0
- added joint velodyne_center_post_arm_to_velodyne_center_joint: type fixed, parent velodyne_center_post_arm_link, child velodyne_center_link, origin xyz=0.04 0 0.05 rpy=0 0 0
- added joint velodyne_center_post_to_velodyne_center_post_arm_joint: type fixed, parent velodyne_center_post_link, child velodyne_center_post_arm_link, origin xyz=0.03 0 0.22675 rpy=0 0 0
- joint base_to_velodyne_front_post_joint: origin xyz=0.63 0.0 1.52325 rpy=0 0 0 -> xyz=1.23 0.0 1.27325 rpy=0 0 0
- joint velodyne_front_post_to_velodyne_front_post_arm_joint: origin xyz=0.03 0 0.22675 rpy=0 0 0 -> xyz=0.03 0 -0.02325 rpy=0 0 0
