Commit message: confiffure URDF

File: urdf/ouxt_wamv.urdf (robot description, URDF)
Before this commit: robot WAM-V, 25 links, 24 joints
Links:
- added link left_camera_link_optical
- added link middle_camera_link_optical
- added link right_camera_link_optical
Joints:
- added joint left_camera_to_left_camera_optical_joint: type fixed, parent left_camera_link, child left_camera_link_optical, origin xyz=0 0 0 rpy=-1.57079632679 0 -1.57079632679
- added joint middle_camera_to_middle_camera_optical_joint: type fixed, parent middle_camera_link, child middle_camera_link_optical, origin xyz=0 0 0 rpy=-1.57079632679 0 -1.57079632679
- added joint right_camera_to_right_camera_optical_joint: type fixed, parent right_camera_link, child right_camera_link_optical, origin xyz=0 0 0 rpy=-1.57079632679 0 -1.57079632679
- joint base_to_left_camera_post_joint: origin xyz=0.7 0.2 1.38475 rpy=0 0 0 -> xyz=0.7 0.4 1.38475 rpy=0 0 2.0944
- joint base_to_right_camera_post_joint: origin xyz=0.7 -0.2 1.38475 rpy=0 0 0 -> xyz=0.7 -0.4 1.38475 rpy=0 0 -2.0944
